File: high_side/control_bdr.sch (EAGLE design)
At the start: 48 parts

Commit message: Rework dirs
Parts:
- removed FAN_1_S1, FAN_1_S2, FAN_1_S3: PIN2F061.040, con-faston:PIN2F061.040
- added CN3: (no value), jst-vh:B5P-VH
- R1, R2, R3, R4: value 330 -> 80
Connections:
- removed net N$31: OK2.A, SV1.1
- new net N$25: OK2.A, SV1.2
- net N$11: now also SV1.6
- net N$2: now also CN3.1; no longer FAN_1_S1.1
- net N$23: now also SV1.7
- net N$27: now also RELAY_FAN1_S21.2; no longer RELAY_FAN1_S31.2
- net N$28: now also RELAY_FAN1_S31.2; no longer RELAY_FAN1_S21.2
- net N$3: now also CN3.5, RELAY_FAN1_S32.S; no longer FAN_1_S2.1, RELAY_FAN1_S22.S
- net N$30: now also SV1.4
- net N$32: now also SV1.3
- net N$33: now also SV1.1
- net N$34: now also SV1.8
- net N$4: now also CN3.3, RELAY_FAN1_S22.S; no longer FAN_1_S3.1, RELAY_FAN1_S32.S
Other:
- moved on the sheet: RELAY_FAN1_S2, RELAY_FAN1_S3
